Commit message: Feat: Integrate EKF sensor fusion with IMU and Odom
- Added IMU sensor plugin to delivery_robot.xacro
- Disabled Gazebo odom TF to prevent conflicts with EKF
- Created ekf.yaml for robot_localization (fusing /odom and /imu)
- Updated navigation.launch.py to start ekf_node with Nav2

File: src/delivery_robot_description/urdf/delivery_robot.xacro (robot description, xacro)
@@ -111,4 +111,10 @@
     <origin xyz="0.13 0 0.02" rpy="0 0 0"/>
   </joint>
+  <link name="imu_link"/>
+  <joint name="imu_joint" type="fixed">
+    <parent link="base_link"/>
+    <child link="imu_link"/>
+    <origin xyz="0 0 0.05" rpy="0 0 0"/>
+  </joint>
   <gazebo reference="base_link"><material>Gazebo/Grey</material></gazebo>
   <gazebo reference="top_plate"><material>Gazebo/White</material></gazebo>
@@ -121,14 +127,15 @@
       <right_joint>front_right_wheel_joint</right_joint>
       <right_joint>rear_right_wheel_joint</right_joint>
-      <wheel_separation>0.245</wheel_separation>
+      <wheel_separation>0.28</wheel_separation>
       <wheel_diameter>0.065</wheel_diameter>
       <max_wheel_torque>5.0</max_wheel_torque>
       <max_wheel_acceleration>1.0</max_wheel_acceleration>
       <publish_odom>true</publish_odom>
-      <publish_odom_tf>true</publish_odom_tf> <publish_wheel_tf>true</publish_wheel_tf>
+      <publish_odom_tf>false</publish_odom_tf> <publish_wheel_tf>true</publish_wheel_tf>
       <odometry_frame>odom</odometry_frame>
       <robot_base_frame>base_footprint</robot_base_frame>
       <command_topic>cmd_vel</command_topic>
       <odometry_topic>odom</odometry_topic>
+      <odometry_source>encoder</odometry_source>
     </plugin>
   </gazebo>
@@ -176,3 +183,16 @@
     <kd>10.0</kd>
   </gazebo>
+  <gazebo reference="imu_link">
+    <sensor name="imu_sensor" type="imu">
+      <plugin name="imu_plugin" filename="libgazebo_ros_imu_sensor.so">
+        <ros>
+          <remapping>~/out:=imu</remapping>
+        </ros>
+        <initial_orientation_as_reference>false</initial_orientation_as_reference>
+      </plugin>
+      <always_on>true</always_on>
+      <update_rate>100</update_rate>
+      <visualize>true</visualize>
+    </sensor>
+  </gazebo>
 </robot>

Commit message: feat: Stable 4-wheel robot simulation with World Odom

File: src/delivery_robot_description/urdf/delivery_robot.xacro (robot description, xacro)
@@ -3,123 +3,188 @@
   <xacro:macro name="box_inertia" params="m w h d">
     <inertial>
-      <origin xyz="0.05 0 0.02" rpy="0 0 0"/>
-      <mass value="${m}"/>
-      <inertia ixx="${(m/12) * (h*h + d*d)}" ixy="0.0" ixz="0.0" iyy="${(m/12) * (w*w + d*d)}" iyz="0.0" izz="${(m/12) * (w*w + h*h)}"/>
+      <origin xyz="0 0 0" rpy="0 0 0" />
+      <mass value="${m}" />
+      <inertia ixx="${(m/12) * (h*h + d*d)}" ixy="0.0" ixz="0.0"
+               iyy="${(m/12) * (w*w + d*d)}" iyz="0.0"
+               izz="${(m/12) * (w*w + h*h)}" />
     </inertial>
   </xacro:macro>
   <xacro:macro name="cylinder_inertia" params="m r h">
     <inertial>
-      <mass value="${m}"/>
-      <inertia ixx="${(m/12) * (3*r*r + h*h)}" ixy="0" ixz="0" iyy="${(m/12) * (3*r*r + h*h)}" iyz="0" izz="${(m/2) * (r*r)}"/>
+      <mass value="${m}" />
+      <inertia ixx="${(m/12) * (3*r*r + h*h)}" ixy="0" ixz="0" iyy="${(m/12) * (3*r*r + h*h)}"
+        iyz="0" izz="${(m/2) * (r*r)}" />
     </inertial>
   </xacro:macro>
-  <link name="base_footprint"/>
+  <link name="base_footprint" />
   <joint name="base_footprint_joint" type="fixed">
-  <parent link="base_footprint"/>
-  <child link="base_link"/>
-  <origin xyz="0 0 0.0325" rpy="0 0 0"/> </joint>
+    <parent link="base_footprint" />
+    <child link="base_link" />
+    <origin xyz="0 0 0.0325" rpy="0 0 0" />
+  </joint>
   <link name="base_link">
     <visual>
-      <geometry><box size="0.297 0.210 0.005"/></geometry>
-      <material name="dark_grey"><color rgba="0.2 0.2 0.2 1"/></material>
+      <geometry>
+        <box size="0.297 0.210 0.005" />
+      </geometry>
+      <material name="dark_grey">
+        <color rgba="0.2 0.2 0.2 1" />
+      </material>
     </visual>
     <collision>
-      <geometry><box size="0.297 0.210 0.005"/></geometry>
+      <geometry>
+        <box size="0.297 0.210 0.005" />
+      </geometry>
     </collision>
-    <xacro:box_inertia m="2.0" w="0.210" h="0.005" d="0.297"/>
+    <xacro:box_inertia m="2.0" w="0.210" h="0.005" d="0.297" />
   </link>
   <xacro:macro name="wheel" params="prefix x_reflect y_reflect">
     <link name="${prefix}_wheel">
       <visual>
-        <origin xyz="0 0 0" rpy="${pi/2} 0 0"/>
-        <geometry><cylinder radius="0.0325" length="0.025"/></geometry>
-        <material name="black"><color rgba="0 0 0 1"/></material>
+        <origin xyz="0 0 0" rpy="${pi/2} 0 0" />
+        <geometry>
+          <cylinder radius="0.0325" length="0.025" />
+        </geometry>
+        <material name="black">
+          <color rgba="0 0 0 1" />
+        </material>
       </visual>
       <collision>
-        <origin xyz="0 0 0" rpy="${pi/2} 0 0"/>
-        <geometry><cylinder radius="0.0325" length="0.025"/></geometry>
+        <origin xyz="0 0 0" rpy="${pi/2} 0 0" />
+        <geometry>
+          <cylinder radius="0.0325" length="0.025" />
+        </geometry>
       </collision>
-      <xacro:cylinder_inertia m="0.1" r="0.0325" h="0.025"/>
+      <xacro:cylinder_inertia m="0.1" r="0.0325" h="0.025" />
     </link>
     <joint name="${prefix}_wheel_joint" type="continuous">
-      <parent link="base_link"/><child link="${prefix}_wheel"/>
-      <origin xyz="${x_reflect*0.1} ${y_reflect*0.12} -0.02" rpy="0 0 0"/>
-      <axis xyz="0 1 0"/>
+      <parent link="base_link" />
+      <child link="${prefix}_wheel" />
+      <origin xyz="${x_reflect*0.1} ${y_reflect*0.12} 0" rpy="0 0 0" />
+      <axis xyz="0 1 0" />
     </joint>
   </xacro:macro>
-  <xacro:wheel prefix="front_left"  x_reflect="1"  y_reflect="1" />
-  <xacro:wheel prefix="front_right" x_reflect="1"  y_reflect="-1" />
-  <xacro:wheel prefix="rear_left"   x_reflect="-1" y_reflect="1" />
-  <xacro:wheel prefix="rear_right"  x_reflect="-1" y_reflect="-1" />
+  <xacro:wheel prefix="front_left" x_reflect="1" y_reflect="1" />
+  <xacro:wheel prefix="front_right" x_reflect="1" y_reflect="-1" />
+  <xacro:wheel prefix="rear_left" x_reflect="-1" y_reflect="1" />
+  <xacro:wheel prefix="rear_right" x_reflect="-1" y_reflect="-1" />
   <link name="top_plate">
     <visual>
-      <geometry><box size="0.297 0.210 0.005"/></geometry>
-      <material name="white"><color rgba="1 1 1 1"/></material>
-    </visual>
-    <collision><geometry><box size="0.297 0.210 0.005"/></geometry></collision>
-    <xacro:box_inertia m="0.4" w="0.210" h="0.005" d="0.297"/>
+      <geometry>
+        <box size="0.297 0.210 0.005" />
+      </geometry>
+      <material name="white">
+        <color rgba="1 1 1 1" />
+      </material>
+    </visual>
+    <collision>
+      <geometry>
+        <box size="0.297 0.210 0.005" />
+      </geometry>
+    </collision>
+    <xacro:box_inertia m="0.4" w="0.210" h="0.005" d="0.297" />
   </link>
   <joint name="top_plate_joint" type="fixed">
-    <parent link="base_link"/><child link="top_plate"/>
-    <origin xyz="0 0 0.1"/>
+    <parent link="base_link" />
+    <child link="top_plate" />
+    <origin xyz="0 0 0.1" />
   </joint>
   <link name="tray_stand">
     <visual>
-      <geometry><cylinder radius="0.01" length="0.05"/></geometry>
-      <material name="grey"><color rgba="0.5 0.5 0.5 1"/></material>
-    </visual>
-    <xacro:cylinder_inertia m="0.1" r="0.01" h="0.05"/>
+      <geometry>
+        <cylinder radius="0.01" length="0.05" />
+      </geometry>
+      <material name="grey">
+        <color rgba="0.5 0.5 0.5 1" />
+      </material>
+    </visual>
+    <xacro:cylinder_inertia m="0.1" r="0.01" h="0.05" />
   </link>
   <joint name="tray_stand_joint" type="fixed">
-    <parent link="top_plate"/><child link="tray_stand"/>
-    <origin xyz="0 0 0.025"/>
+    <parent link="top_plate" />
+    <child link="tray_stand" />
+    <origin xyz="0 0 0.025" />
   </joint>
   <link name="tray_link">
     <visual>
-      <geometry><box size="0.25 0.20 0.005"/></geometry>
-      <material name="grey"><color rgba="0.5 0.5 0.5 1"/></material>
-    </visual>
-    <xacro:box_inertia m="0.2" w="0.20" h="0.005" d="0.25"/>
+      <geometry>
+        <box size="0.25 0.20 0.005" />
+      </geometry>
+      <material name="grey">
+        <color rgba="0.5 0.5 0.5 1" />
+      </material>
+    </visual>
+    <xacro:box_inertia m="0.2" w="0.20" h="0.005" d="0.25" />
   </link>
   <joint name="tray_joint" type="fixed">
-    <parent link="tray_stand"/><child link="tray_link"/>
-    <origin xyz="0 0 0.025"/>
+    <parent link="tray_stand" />
+    <child link="tray_link" />
+    <origin xyz="0 0 0.025" />
   </joint>
   <link name="payload_link">
     <visual>
-      <origin xyz="0 0 0.05"/>
-      <geometry><box size="0.15 0.15 0.1"/></geometry>
-      <material name="blue"><color rgba="0 0 0.8 1"/></material>
-    </visual>
-    <xacro:box_inertia m="1.5" w="0.15" h="0.1" d="0.15"/>
+      <origin xyz="0 0 0.05" />
+      <geometry>
+        <box size="0.15 0.15 0.1" />
+      </geometry>
+      <material name="blue">
+        <color rgba="0 0 0.8 1" />
+      </material>
+    </visual>
+    <xacro:box_inertia m="1.5" w="0.15" h="0.1" d="0.15" />
   </link>
   <joint name="payload_joint" type="fixed">
-    <parent link="tray_link"/><child link="payload_link"/>
-    <origin xyz="0 0 0.005"/>
+    <parent link="tray_link" />
+    <child link="payload_link" />
+    <origin xyz="0 0 0.005" />
   </joint>
   <link name="lidar_link">
     <visual>
-      <geometry><cylinder radius="0.035" length="0.04"/></geometry>
-      <material name="black"><color rgba="0 0 0 1"/></material> </visual>
+      <geometry>
+        <cylinder radius="0.035" length="0.04" />
+      </geometry>
+      <material name="black">
+        <color rgba="0 0 0 1" />
+      </material>
+    </visual>
     <collision>
-      <geometry><cylinder radius="0.035" length="0.04"/></geometry>
+      <geometry>
+        <cylinder radius="0.035" length="0.04" />
+      </geometry>
     </collision>
-    <xacro:cylinder_inertia m="0.15" r="0.035" h="0.04"/>
+    <xacro:cylinder_inertia m="0.15" r="0.035" h="0.04" />
   </link>
   <joint name="lidar_joint" type="fixed">
-    <parent link="top_plate"/><child link="lidar_link"/>
-    <origin xyz="0.13 0 0.02" rpy="0 0 0"/>
-  </joint>
-  <link name="imu_link"/>
+    <parent link="top_plate" />
+    <child link="lidar_link" />
+    <origin xyz="0.13 0 0.02" rpy="0 0 0" />
+  </joint>
+  <link name="imu_link">
+    <inertial>
+      <mass value="0.01" />
+      <origin xyz="0 0 0" rpy="0 0 0" />
+      <inertia ixx="1e-7" ixy="0" ixz="0" iyy="1e-7" iyz="0" izz="1e-7" />
+    </inertial>
+  </link>
   <joint name="imu_joint" type="fixed">
-    <parent link="base_link"/>
-    <child link="imu_link"/>
-    <origin xyz="0 0 0.05" rpy="0 0 0"/>
-  </joint>
-  <gazebo reference="base_link"><material>Gazebo/Grey</material></gazebo>
-  <gazebo reference="top_plate"><material>Gazebo/White</material></gazebo>
-  <gazebo reference="payload_link"><material>Gazebo/Blue</material></gazebo>
+    <parent link="base_link" />
+    <child link="imu_link" />
+    <origin xyz="0 0 0.05" rpy="0 0 0" />
+  </joint>
+  <gazebo reference="base_link">
+    <material>Gazebo/Grey</material>
+  </gazebo>
+  <gazebo reference="top_plate">
+    <material>Gazebo/White</material>
+  </gazebo>
+  <gazebo reference="payload_link">
+    <material>Gazebo/Blue</material>
+  </gazebo>
   <gazebo>
     <plugin name="skid_steer" filename="libgazebo_ros_diff_drive.so">
+      <publish_odom_tf>true</publish_odom_tf>
+      <publish_wheel_tf>true</publish_wheel_tf>
+      <publish_odom>true</publish_odom>
+      <odometry_source>1</odometry_source>
       <num_wheel_pairs>2</num_wheel_pairs>
       <left_joint>front_left_wheel_joint</left_joint>
@@ -127,15 +192,13 @@
       <right_joint>front_right_wheel_joint</right_joint>
       <right_joint>rear_right_wheel_joint</right_joint>
-      <wheel_separation>0.28</wheel_separation>
+      <wheel_separation>0.4</wheel_separation>
       <wheel_diameter>0.065</wheel_diameter>
-      <max_wheel_torque>5.0</max_wheel_torque>
-      <max_wheel_acceleration>1.0</max_wheel_acceleration>
-      <publish_odom>true</publish_odom>
-      <publish_odom_tf>false</publish_odom_tf> <publish_wheel_tf>true</publish_wheel_tf>
+      <max_wheel_torque>100.0</max_wheel_torque>
+      <max_wheel_acceleration>5.0</max_wheel_acceleration>
+      <command_topic>cmd_vel</command_topic>
+      <odometry_topic>odom</odometry_topic>
       <odometry_frame>odom</odometry_frame>
       <robot_base_frame>base_footprint</robot_base_frame>
-      <command_topic>cmd_vel</command_topic>
-      <odometry_topic>odom</odometry_topic>
-      <odometry_source>encoder</odometry_source>
+      <update_rate>50</update_rate>
     </plugin>
   </gazebo>
@@ -145,13 +208,21 @@
       <update_rate>10</update_rate>
       <ray>
-        <scan><horizontal><samples>360</samples><min_angle>-3.14</min_angle><max_angle>3.14</max_angle></horizontal></scan>
+        <scan>
+          <horizontal>
+            <samples>360</samples>
+            <min_angle>-3.14</min_angle>
+            <max_angle>3.14</max_angle>
+          </horizontal>
+        </scan>
         <range>
-        <min>0.20</min>
-        <max>10.0</max>
-        <resolution>0.01</resolution>
+          <min>0.20</min>
+          <max>10.0</max>
+          <resolution>0.01</resolution>
         </range>
       </ray>
       <plugin name="gazebo_ros_lidar" filename="libgazebo_ros_ray_sensor.so">
-        <ros><remapping>~/out:=scan</remapping></ros>
+        <ros>
+          <remapping>~/out:=scan</remapping>
+        </ros>
         <output_type>sensor_msgs/LaserScan</output_type>
         <frame_name>lidar_link</frame_name>
@@ -160,27 +231,28 @@
   </gazebo>
   <gazebo reference="front_left_wheel">
-    <mu1>0.1</mu1>
-    <mu2>0.1</mu2>
+    <mu1>0.5</mu1>
+    <mu2>0.5</mu2>
     <kp>1000000.0</kp>
-    <kd>10.0</kd>
+    <kd>100.0</kd>
   </gazebo>
   <gazebo reference="front_right_wheel">
-    <mu1>0.1</mu1>
-    <mu2>0.1</mu2>
+    <mu1>0.5</mu1>
+    <mu2>0.5</mu2>
     <kp>1000000.0</kp>
-    <kd>10.0</kd>
+    <kd>100.0</kd>
   </gazebo>
   <gazebo reference="rear_left_wheel">
-    <mu1>0.1</mu1>
-    <mu2>0.1</mu2>
+    <mu1>0.0</mu1>
+    <mu2>0.0</mu2>
     <kp>1000000.0</kp>
-    <kd>10.0</kd>
+    <kd>100.0</kd>
   </gazebo>
   <gazebo reference="rear_right_wheel">
-    <mu1>0.1</mu1>
-    <mu2>0.1</mu2>
+    <mu1>0.0</mu1>
+    <mu2>0.0</mu2>
     <kp>1000000.0</kp>
-    <kd>10.0</kd>
-  </gazebo>
+    <kd>100.0</kd>
+  </gazebo>
+  <!--
   <gazebo reference="imu_link">
     <sensor name="imu_sensor" type="imu">
@@ -188,11 +260,55 @@
         <ros>
           <remapping>~/out:=imu</remapping>
+          <namespace>/</namespace>
         </ros>
-        <initial_orientation_as_reference>false</initial_orientation_as_reference>
-      </plugin>
+        <initial_orientation_as_reference>true</initial_orientation_as_reference>
+        <frame_name>imu_link</frame_name> </plugin>
       <always_on>true</always_on>
       <update_rate>100</update_rate>
       <visualize>true</visualize>
+      <imu>
+        <angular_velocity>
+          <x>
+            <noise type="gaussian">
+              <mean>0.0</mean>
+              <stddev>0.0002</stddev>
+            </noise>
+          </x>
+          <y>
+            <noise type="gaussian">
+              <mean>0.0</mean>
+              <stddev>0.0002</stddev>
+            </noise>
+          </y>
+          <z>
+            <noise type="gaussian">
+              <mean>0.0</mean>
+              <stddev>0.0002</stddev>
+            </noise>
+          </z>
+        </angular_velocity>
+        <linear_acceleration>
+          <x>
+            <noise type="gaussian">
+              <mean>0.0</mean>
+              <stddev>0.017</stddev>
+            </noise>
+          </x>
+          <y>
+            <noise type="gaussian">
+              <mean>0.0</mean>
+              <stddev>0.017</stddev>
+            </noise>
+          </y>
+          <z>
+            <noise type="gaussian">
+              <mean>0.0</mean>
+              <stddev>0.017</stddev>
+            </noise>
+          </z>
+        </linear_acceleration>
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